File: hardware/kelvindmmwifi.sch (KiCad schematic (older format))
At the start: 18 parts, among them P1 IN+, P2 IN-, P3 V+, P4 OUT, P5 GND, P6 3V3, P7 ADC, P8 PGM_ETC, U1 COMP-MIC7721, U2 AP1117

Commit message: update with current design etc.
Other:
- note added: "Reference on DMM to IN-\nBUFF? to IN+"
Changed lines of the file:
@@
 	0    1    1    0
 $EndComp
+Text Notes 2200 1150 0    60   ~ 0
+Reference on DMM to IN-\nBUFF?  to IN+
 $EndSCHEMATC
